File: triton-delay.sch (KiCad schematic (older format))
At the start: 58 parts, among them IC1 PT2399, IC2 TL072, J1 Stomp_Connector, J2 Power_Connector, SW1 Time

Commit message: v2-3_2: tied unused leg 1 of Slow B10k to wiper, moved a few traces for better ground plane coverage
Connections:
- wire segments 188 -> 191
Changed lines of the file:
@@
 Connection ~ 2175 4725
 Connection ~ 2750 3975
+Connection ~ 2775 5075
 Wire Wire Line
 	1925 4475 2175 4475
@@
 	2650 3975 2750 3975
 Wire Wire Line
-	2725 5075 2800 5075
+	2725 5075 2775 5075
 Wire Wire Line
 	2750 2475 2750 2575
@@
 	2750 3975 2850 3975
 Wire Wire Line
+	2775 5075 2800 5075
+Wire Wire Line
+	2775 5225 2775 5075
+Wire Wire Line
 	2850 3425 2850 3575
 Wire Wire Line
@@
 	2950 4925 2950 4850
 Wire Wire Line
+	2950 5225 2775 5225
+Wire Wire Line
 	3300 6550 3550 6550

Commit message: v2-3_2: tied unused leg 1 of Slow B10k to wiper, moved a few traces for better ground plane coverage
Other:
- note added: "triton-delay v2-3_2"
- note removed: "triton-delay v2-3_1"
Changed lines of the file:
@@
 	9075 5075 9075 5425
 Text Notes 8225 7500 2    50   ~ 0
-triton-delay v2-3_1
+triton-delay v2-3_2
 Text Notes 8250 6750 2    100  ~ 0
 TRITON DELAY
