File: triton-delay.kicad_pcb (KiCad board)
At the start: 2 copper layers, 52.3 x 47.8 mm, 58 parts, among them IC1 PT2399, IC2 TL072, J1 Stomp_Connector, J2 Power_Connector, SW1 Time

Commit message: v2-3_2: tied unused leg 1 of Slow B10k to wiper, moved a few traces for better ground plane coverage
Connections:
- RV3 pad 2: Net-(RV3-Pad2) -> Net-(RV3-Pad1)
- SW1 pad 2: Net-(RV3-Pad2) -> Net-(RV3-Pad1)
Routing:
- net Net-(RV3-Pad1): track 0.00 -> 56.8 mm
- net Net-(RV3-Pad2): track 48.0 -> 0.00 mm
- net Net-(C18-Pad1): track 28.1 -> 13.4 mm
- net Net-(C8-Pad2): track 12.2 -> 19.0 mm
- net Net-(R12-Pad2): track 38.9 -> 42.8 mm
- net Net-(C15-Pad1): track 40.9 -> 37.9 mm
- net Net-(C8-Pad1): track 18.6 -> 21.0 mm
- net Net-(C11-Pad2): track 37.7 -> 40.1 mm
- net VA: track 63.3 -> 65.6 mm
- net Net-(C6-Pad2): track 39.0 -> 40.6 mm
- net Net-(C20-Pad1): track 23.9 -> 23.0 mm
- net Net-(C13-Pad1): track 23.2 -> 23.8 mm
Other:
- board text added: "v2-3_2 2020-03-27"
- board text removed: "v2-3_1 2020-03-27"

Commit message: updated to KiCad 6.0
Other:
- net class Default removed
